Commit message: u

File: gazebo/gz_rrbot.xacro (robot description, xacro)
@@ -37,5 +37,5 @@
   <gazebo>
     <plugin name="gz_ros2_control" filename="libgazebo_ros2_control.so">
-      <parameters>$(find robot_gazebo)/config/rrbot_gazebo_forward_controller_position.yaml</parameters>
+      <parameters>$(find rrbot)/config/rrbot_gazebo_forward_controller_position.yaml</parameters>
     </plugin>
   </gazebo>

File: xacro/rrbot.xacro (robot description, xacro)
@@ -6,5 +6,5 @@
 <!-- *********************************************************************************************************************************  -->
 <!-- ****************************************************** Parameters ***************************************************************  -->
-  <xacro:property name="mesh_path"      value="package://robot_gazebo/meshes/rrbot/" />
+  <xacro:property name="mesh_path"      value="package://rrbot/meshes/rrbot/" />
   <xacro:property name="name_space"     value="rrbot" />
   <xacro:property name="prefix"         value=""      />
@@ -32,7 +32,7 @@
   <xacro:property name="tool_z"         value="${height3}" />
 <!-- ****************************************************** Includes *****************************************************************  -->
-  <xacro:include filename="$(find robot_gazebo)/xacro/common_rviz_materials.xacro" />   <!-- RVIZ Colors                                -->
-  <xacro:include filename="$(find robot_gazebo)/gazebo/gz_rrbot.xacro" />               <!--  Gazebo                                    -->
-  <xacro:include filename="$(find robot_gazebo)/ros2_control/r2c_rrbot.xacro" />        <!--  ROS2_Control                              -->
+  <xacro:include filename="$(find rrbot)/xacro/common_rviz_materials.xacro" />   <!-- RVIZ Colors                                -->
+  <xacro:include filename="$(find rrbot)/gazebo/gz_rrbot.xacro" />               <!--  Gazebo                                    -->
+  <xacro:include filename="$(find rrbot)/ros2_control/r2c_rrbot.xacro" />        <!--  ROS2_Control                              -->
 <!-- ****************************************************** Base Joint ***************************************************************  -->
   <joint name="${prefix}base_joint" type="fixed">

Commit message: u

File: gazebo/gz_rrbot.xacro (robot description, xacro)
@@ -7,24 +7,16 @@
 <!-- ****************************************************** Base Link ****************************************************************  -->
   <gazebo reference="${prefix}base">
-      <mu1>0.2</mu1>
-      <mu2>0.2</mu2>
       <material>Gazebo/Orange</material>
   </gazebo>
 <!-- ****************************************************** Link 1 *******************************************************************  -->
   <gazebo reference="${prefix}link2">
-      <mu1>0.2</mu1>
-      <mu2>0.2</mu2>
       <material>Gazebo/Orange</material>
   </gazebo>
 <!-- ****************************************************** Link 2 *******************************************************************  -->
   <gazebo reference="${prefix}link3">
-      <mu1>0.2</mu1>
-      <mu2>0.2</mu2>
       <material>Gazebo/Orange</material>
   </gazebo>
 <!-- ****************************************************** Camera Link **************************************************************  -->
   <gazebo reference="${prefix}camera">
-      <mu1>0.2</mu1>
-      <mu2>0.2</mu2>
       <material>Gazebo/Green</material>
   </gazebo>
@@ -34,110 +26,4 @@
     <static>true</static>
   </gazebo>
-<!-- ****************************************************** ROS Control Plugin *******************************************************  -->
-  <gazebo>
-    <plugin name="gz_ros2_control" filename="libgazebo_ros2_control.so">
-      <parameters>$(find robot_gazebo)/config/rrbot_gazebo_forward_controller_position.yaml</parameters>
-    </plugin>
-  </gazebo>
-<!-- ******************************************************  Joint States Publisher **************************************************  -->
-  <gazebo>
-    <plugin name="joint_states_pub" filename="libgazebo_ros_joint_state_publisher.so">
-      <ros>
-        <namespace>${name_space}</namespace>
-      </ros>
-      <joint_name>${prefix}base_joint</joint_name>
-      <joint_name>${prefix}joint1</joint_name>
-      <joint_name>${prefix}joint2</joint_name>
-      <update_rate>100.0</update_rate>
-    </plugin>
- </gazebo>
-<!-- ******************************************************  Camera ******************************************************************  -->
-  <gazebo reference="${prefix}camera">
-    <sensor type="camera" name="camera">
-      <update_rate>30.0</update_rate>
-      <camera name="head">
-        <horizontal_fov>${radians(80)}</horizontal_fov>
-        <image>
-          <width>1280</width>
-          <height>720</height>
-          <format>R8G8B8</format>
-        </image>
-        <clip>
-          <near>0.02</near>
-          <far>300</far>
-        </clip>
-        <noise>
-          <type>gaussian</type>
-          <!-- Noise is sampled independently per pixel on each frame.
-          That pixel's noise value is added to each of its color
-          channels, which at that point lie in the range [0,1]. -->
-          <mean>0.0</mean>
-          <stddev>0.007</stddev>
-        </noise>
-      </camera>
-      <plugin name="camera_controller" filename="libgazebo_ros_camera.so">
-        <ros>
-          <namespace>${name_space}</namespace>
-        </ros>
-        <alwaysOn>true</alwaysOn>
-        <updateRate>0.0</updateRate>
-        <cameraName>camera</cameraName>
-        <imageTopicName>image_raw</imageTopicName>
-        <cameraInfoTopicName>camera_info</cameraInfoTopicName>
-        <frameName>camera_optical</frameName>
-        <!-- setting hackBaseline to anything but 0.0 will cause a misalignment
-        between the gazebo sensor image and the frame it is supposed to
-        be attached to -->
-        <hackBaseline>0.0</hackBaseline>
-        <distortionK1>0.0</distortionK1>
-        <distortionK2>0.0</distortionK2>
-        <distortionK3>0.0</distortionK3>
-        <distortionT1>0.0</distortionT1>
-        <distortionT2>0.0</distortionT2>
-        <CxPrime>0</CxPrime>
-        <Cx>0.0</Cx>
-        <Cy>0.0</Cy>
-        <focalLength>0.0</focalLength>
-      </plugin>
-    </sensor>
-    <material>Gazebo/Green</material>
-  </gazebo>
-<!-- ****************************************************** hokuyo  ******************************************************************  -->
-  <gazebo reference="${prefix}hokuyo">
-    <sensor type="ray" name="head_hokuyo_sensor">
-      <plugin name="hokuyo" filename="libgazebo_ros_ray_sensor.so">
-        <ros>
-          <namespace>${name_space}</namespace>
-        </ros>
-        <output_type>sensor_msgs/LaserScan</output_type>
-      </plugin>
-      <update_rate>30</update_rate>
-      <pose>0 0 0 0 0 0</pose>
-      <visualize>false</visualize>
-      <ray>
-        <scan>
-          <horizontal>
-            <samples>720</samples>
-            <resolution>1</resolution>
-            <min_angle>-${radians(180)}</min_angle>
-            <max_angle> ${radians(180)}</max_angle>
-          </horizontal>
-        </scan>
-        <range>
-          <min>0.10</min>
-          <max>30.0</max>
-          <resolution>0.01</resolution>
-        </range>
-<!-- Noise parameters based on published spec for Hokuyo laser achieving "+-30mm" accuracy at range < 10m.  A mean of 0.0m and stddev   -->
-<!-- of 0.01m will put 99.7% of samples within 0.03m of the true reading.                                                               -->
-        <noise>
-          <type>gaussian</type>
-          <mean>0.0</mean>
-          <stddev>0.01</stddev>
-        </noise>
-      </ray>
-    </sensor>
-    <!-- <material>Gazebo/Red</material> -->
-  </gazebo>
 <!-- ****************************************************** END **********************************************************************  -->
 </robot>

Commit message: u

File: gazebo/gz_rrbot.xacro (robot description, xacro)
@@ -7,16 +7,24 @@
 <!-- ****************************************************** Base Link ****************************************************************  -->
   <gazebo reference="${prefix}base">
+      <mu1>0.2</mu1>
+      <mu2>0.2</mu2>
       <material>Gazebo/Orange</material>
   </gazebo>
 <!-- ****************************************************** Link 1 *******************************************************************  -->
   <gazebo reference="${prefix}link2">
+      <mu1>0.2</mu1>
+      <mu2>0.2</mu2>
       <material>Gazebo/Orange</material>
   </gazebo>
 <!-- ****************************************************** Link 2 *******************************************************************  -->
   <gazebo reference="${prefix}link3">
+      <mu1>0.2</mu1>
+      <mu2>0.2</mu2>
       <material>Gazebo/Orange</material>
   </gazebo>
 <!-- ****************************************************** Camera Link **************************************************************  -->
   <gazebo reference="${prefix}camera">
+      <mu1>0.2</mu1>
+      <mu2>0.2</mu2>
       <material>Gazebo/Green</material>
   </gazebo>
@@ -26,4 +34,73 @@
     <static>true</static>
   </gazebo>
+<!-- ****************************************************** ROS Control Plugin *******************************************************  -->
+  <gazebo>
+    <plugin name="gz_ros2_control" filename="libgazebo_ros2_control.so">
+      <parameters>$(find robot_gazebo)/config/rrbot_forward_position.yaml</parameters>
+    </plugin>
+  </gazebo>
+<!-- ******************************************************  Joint States Publisher **************************************************  -->
+  <gazebo>
+    <plugin name="joint_states_pub" filename="libgazebo_ros_joint_state_publisher.so">
+      <ros>
+        <namespace>${name_space}</namespace>
+      </ros>
+      <joint_name>${prefix}base_joint</joint_name>
+      <joint_name>${prefix}joint1</joint_name>
+      <joint_name>${prefix}joint2</joint_name>
+      <update_rate>100.0</update_rate>
+    </plugin>
+ </gazebo>
+<!-- ******************************************************  Camera ******************************************************************  -->
+  <gazebo reference="${prefix}camera">
+    <sensor type="camera" name="camera">
+      <update_rate>30.0</update_rate>
+      <camera name="head">
+        <horizontal_fov>${radians(80)}</horizontal_fov>
+        <image>
+          <width>1280</width>
+          <height>720</height>
+          <format>R8G8B8</format>
+        </image>
+        <clip>
+          <near>0.02</near>
+          <far>300</far>
+        </clip>
+        <noise>
+          <type>gaussian</type>
+          <!-- Noise is sampled independently per pixel on each frame.
+          That pixel's noise value is added to each of its color
+          channels, which at that point lie in the range [0,1]. -->
+          <mean>0.0</mean>
+          <stddev>0.007</stddev>
+        </noise>
+      </camera>
+      <plugin name="camera_controller" filename="libgazebo_ros_camera.so">
+        <ros>
+          <namespace>${name_space}</namespace>
+        </ros>
+        <alwaysOn>true</alwaysOn>
+        <updateRate>0.0</updateRate>
+        <cameraName>camera</cameraName>
+        <imageTopicName>image_raw</imageTopicName>
+        <cameraInfoTopicName>camera_info</cameraInfoTopicName>
+        <frameName>camera_optical</frameName>
+        <!-- setting hackBaseline to anything but 0.0 will cause a misalignment
+        between the gazebo sensor image and the frame it is supposed to
+        be attached to -->
+        <hackBaseline>0.0</hackBaseline>
+        <distortionK1>0.0</distortionK1>
+        <distortionK2>0.0</distortionK2>
+        <distortionK3>0.0</distortionK3>
+        <distortionT1>0.0</distortionT1>
+        <distortionT2>0.0</distortionT2>
+        <CxPrime>0</CxPrime>
+        <Cx>0.0</Cx>
+        <Cy>0.0</Cy>
+        <focalLength>0.0</focalLength>
+      </plugin>
+    </sensor>
+    <material>Gazebo/Green</material>
+  </gazebo>
 <!-- ****************************************************** END **********************************************************************  -->
 </robot>

File: xacro/rrbot copy.xacro (robot description, xacro)
@@ -34,5 +34,5 @@
   <xacro:include filename="$(find rrbot)/xacro/common_rviz_materials.xacro" />   <!--  RVIZ Colors                               -->
   <xacro:include filename="$(find rrbot)/gazebo/gz_rrbot.xacro" />               <!--  Gazebo                                    -->
-  <xacro:include filename="$(find rrbot)/ros2_control/r2c_rrbot.xacro" />        <!--  ROS2_Control                              -->
+  <!-- <xacro:include filename="$(find rrbot)/ros2_control/r2c_rrbot.xacro" />         ROS2_Control                              -->
 <!-- ****************************************************** Base Joint ***************************************************************  -->
   <joint name="${prefix}base_joint" type="fixed">
@@ -176,4 +176,31 @@
 <!-- ****************************************************** Camera Optical Link ******************************************************  -->
   <link name="${prefix}camera_optical"/>
+<!-- ****************************************************** Hokuyo Joint *************************************************************  -->
+  <joint name="${prefix}hokuyo_joint" type="fixed">
+    <axis xyz="0 1 0" />
+    <origin xyz="0 0 ${hokuyo_z}" rpy="0 0 0"/>
+    <parent link="${prefix}link3"/>
+    <child link="${prefix}hokuyo"/>
+  </joint>
+<!-- ****************************************************** Hokuyo Link **************************************************************  -->
+  <link name="${prefix}hokuyo">
+    <collision>
+      <origin xyz="0 0 0" rpy="0 0 0"/>
+      <geometry>
+        <mesh filename="${mesh_path}hokuyo.dae"/> <!--  <box size="${hokuyo_length} ${hokuyo_width} ${hokuyo_height}"/> -->
+      </geometry>
+    </collision>
+    <visual>
+      <origin xyz="0 0 0" rpy="0 0 0"/>
+      <geometry>
+        <mesh filename="${mesh_path}hokuyo.dae"/> <!--  <box size="${hokuyo_length} ${hokuyo_width} ${hokuyo_height}"/> -->
+      </geometry>
+    </visual>
+    <inertial>
+      <mass value="${hokuyo_mass}" />
+      <origin xyz="0 0 0" rpy="0 0 0"/>
+      <inertia ixx="1e-6" ixy="0" ixz="0" iyy="1e-6" iyz="0" izz="1e-6" />
+    </inertial>
+  </link>
 <!-- ****************************************************** END **********************************************************************  -->
 </robot>
