Commit message: u

File: xacro/rrbot.xacro (robot description, xacro)
@@ -6,174 +6,14 @@
 <!-- *********************************************************************************************************************************  -->
 <!-- ****************************************************** Parameters ***************************************************************  -->
-  <xacro:property name="mesh_path"      value="package://rrbot/meshes/rrbot/" />
-  <xacro:property name="name_space"     value="rrbot" />
-  <xacro:property name="prefix"         value=""      />
-  <xacro:property name="mass"           value="1"                       /> <!-- arbitrary value for mass -->
-  <xacro:property name="width"          value="0.1"                     /> <!-- Square dimensions (widthxwidth) of beams -->
-  <xacro:property name="height1"        value="2"                       /> <!-- Link 1 (Base) -->
-  <xacro:property name="height2"        value="1"                       /> <!-- Link 2 -->
-  <xacro:property name="height3"        value="1"                       /> <!-- Link 3 -->
-  <xacro:property name="joint_gap"      value="0.05"                    /> <!-- Space btw top of beam and the each joint -->
-  <xacro:property name="joint1_y"       value="${width}"                />
-  <xacro:property name="joint1_z"       value="${height1-joint_gap}"    />
-  <xacro:property name="joint2_y"       value="${width}"                />
-  <xacro:property name="joint2_z"       value="${height2-joint_gap*2}"  />
-  <xacro:property name="camera_mass"    value="1e-5"     />
-  <xacro:property name="camera_width"   value="0.05"     />
-  <xacro:property name="camera_length"  value="0.05"     />
-  <xacro:property name="camera_height"  value="0.05"     />
-  <xacro:property name="camera_x"       value="${(width+camera_width)/2}" />
-  <xacro:property name="camera_z"       value="${height3-joint_gap*2}" />
-  <xacro:property name="hokuyo_mass"    value="1e-5"     />
-  <xacro:property name="hokuyo_width"   value="0.05"     />
-  <xacro:property name="hokuyo_length"  value="0.05"     />
-  <xacro:property name="hokuyo_height"  value="0.0706"   />
-  <xacro:property name="hokuyo_z"       value="${height3-joint_gap/2}" />
-  <xacro:property name="tool_z"         value="${height3}" />
+    <xacro:property name="pkg_path"     value="$(find rrbot)"           />
+    <xacro:property name="mesh_path"    value="${pkg_path}/meshes/"     />
+    <xacro:property name="xacro_path"   value="${pkg_path}/xacro/"      />
+    <xacro:property name="name_space"   value="rrbot" />
+    <xacro:property name="prefix"       value=""      />
 <!-- ****************************************************** Includes *****************************************************************  -->
-  <xacro:include filename="$(find rrbot)/xacro/common_rviz_materials.xacro" />   <!--  RVIZ Colors                               -->
-  <xacro:include filename="$(find rrbot)/gazebo/gz_rrbot.xacro" />               <!--  Gazebo                                    -->
-  <xacro:include filename="$(find rrbot)/ros2_control/r2c_rrbot.xacro" />        <!--  ROS2_Control                              -->
-<!-- ****************************************************** Base Joint ***************************************************************  -->
-  <joint name="${prefix}base_joint" type="fixed">
-    <origin xyz="0 0 0" rpy="0 0 0" />
-    <parent link="world"/>
-    <child link="${prefix}base" />
-  </joint>
-<!-- ****************************************************** Base Link ****************************************************************  -->
-  <link name="${prefix}base">
-    <collision>
-      <origin xyz="0 0 ${height1/2}" rpy="0 0 0"/>
-      <geometry>
-        <box size="${width} ${width} ${height1}"/>
-      </geometry>
-    </collision>
-    <visual>
-      <origin xyz="0 0 ${height1/2}" rpy="0 0 0"/>
-      <geometry>
-        <box size="${width} ${width} ${height1}"/>
-      </geometry>
-      <material name="orange"/>
-    </visual>
-    <inertial>
-      <origin xyz="0 0 ${height1/2}" rpy="0 0 0"/>
-      <mass value="${mass}"/>
-      <inertia
-        ixx="${mass / 12.0 * (width*width + height1*height1)}" ixy="0.0" ixz="0.0"
-        iyy="${mass / 12.0 * (height1*height1 + width*width)}" iyz="0.0"
-        izz="${mass / 12.0 * (width*width + width*width)}"/>
-    </inertial>
-  </link>
-<!-- ****************************************************** Joint 1 ******************************************************************  -->
-  <joint name="${prefix}joint1" type="continuous">
-    <parent link="${prefix}base"/>
-    <child link="${prefix}link2"/>
-    <origin xyz="0 ${joint1_y} ${joint1_z}" rpy="0 0 0"/>
-    <axis xyz="0 1 0"/>
-    <dynamics damping="0.7"/>
-  </joint>
-<!-- ****************************************************** Link 2 *******************************************************************  -->
-  <link name="${prefix}link2">
-    <collision>
-      <origin xyz="0 0 ${height2/2 - joint_gap}" rpy="0 0 0"/>
-      <geometry>
-        <box size="${width} ${width} ${height2}"/>
-      </geometry>
-    </collision>
-    <visual>
-      <origin xyz="0 0 ${height2/2 - joint_gap}" rpy="0 0 0"/>
-      <geometry>
-        <box size="${width} ${width} ${height2}"/>
-      </geometry>
-      <material name="yellow"/>
-    </visual>
-    <inertial>
-      <origin xyz="0 0 ${height2/2 - joint_gap}" rpy="0 0 0"/>
-      <mass value="${mass}"/>
-      <inertia
-        ixx="${mass / 12.0 * (width*width + height2*height2)}" ixy="0.0" ixz="0.0"
-        iyy="${mass / 12.0 * (height2*height2 + width*width)}" iyz="0.0"
-        izz="${mass / 12.0 * (width*width + width*width)}"/>
-    </inertial>
-  </link>
-<!-- ****************************************************** Joint 2 ******************************************************************  -->
-  <joint name="${prefix}joint2" type="continuous">
-    <parent link="${prefix}link2"/>
-    <child link="${prefix}link3"/>
-    <origin xyz="0 ${joint2_y} ${joint2_z}" rpy="0 0 0"/>
-    <axis xyz="0 1 0"/>
-    <dynamics damping="0.7"/>
-  </joint>
-<!-- ****************************************************** Link 3 *******************************************************************  -->
-  <link name="${prefix}link3">
-    <collision>
-      <origin xyz="0 0 ${height3/2 - joint_gap}" rpy="0 0 0"/>
-      <geometry>
-        <box size="${width} ${width} ${height3}"/>
-      </geometry>
-    </collision>
-    <visual>
-      <origin xyz="0 0 ${height3/2 - joint_gap}" rpy="0 0 0"/>
-      <geometry>
-        <box size="${width} ${width} ${height3}"/>
-      </geometry>
-      <material name="orange"/>
-    </visual>
-    <inertial>
-      <origin xyz="0 0 ${height3/2 - joint_gap}" rpy="0 0 0"/>
-      <mass value="${mass}"/>
-      <inertia
-        ixx="${mass / 12.0 * (width*width + height3*height3)}" ixy="0.0" ixz="0.0"
-        iyy="${mass / 12.0 * (height3*height3 + width*width)}" iyz="0.0"
-        izz="${mass / 12.0 * (width*width + width*width)}"/>
-    </inertial>
-  </link>
-<!-- ****************************************************** Tool Joint ***************************************************************  -->
-  <joint name="${prefix}tool_joint" type="fixed">
-    <origin xyz="0 0 ${tool_z}" rpy="0 0 0" />
-    <parent link="${prefix}link3"/>
-    <child link="${prefix}tool" />
-  </joint>
-<!-- ****************************************************** Tool Link ****************************************************************  -->
-  <link name="${prefix}tool" />
-<!-- ****************************************************** Camera Joint *************************************************************  -->
-  <joint name="${prefix}camera_joint" type="fixed">
-    <axis xyz="0 1 0" />
-    <origin xyz="${camera_x} 0 ${camera_z}" rpy="0 0 0"/>
-    <parent link="${prefix}link3"/>
-    <child link="${prefix}camera"/>
-  </joint>
-<!-- ****************************************************** Camera Link **************************************************************  -->
-<link name="${prefix}camera">
-  <inertial>
-    <mass value="${camera_mass}"/>
-    <origin xyz="0 0 0" rpy=" 0 0 0"/>
-    <inertia ixx="1e-6" ixy="0" ixz="0" iyy="1e-6" iyz="0" izz="1e-6" />
-  </inertial>
-  <visual name="camera_visual">
-    <origin xyz="0 0 0" rpy="0 0 0" />
-    <geometry>
-      <box size="${camera_length} ${camera_width} ${camera_height}"/>
-    </geometry>
-    <material name="green"/>
-  </visual>
-  <collision name="camera_colision">
-    <origin xyz="0 0 0" rpy="0 0 0" />
-    <geometry>
-      <box size="${camera_length} ${camera_width} ${camera_height}"/>
-    </geometry>
-  </collision>
-</link>
-<!-- ****************************************************** Camera Optical Joint *****************************************************  -->
-<!-- generate an optical frame http://www.ros.org/reps/rep-0103.html#suffix-frames so that ros and opencv can operate on the camera     -->
-<!-- frame correctly. these values have to be these values otherwise the gazebo camera image won't be aligned properly with the frame   -->
-<!-- it is supposedly originating from                                                                                                  -->
-  <joint name="${prefix}camera_optical_joint" type="fixed">
-    <origin xyz="0 0 0" rpy="${-radians(90)} 0 ${-radians(90)}"/>
-    <parent link="${prefix}camera"/>
-    <child link="${prefix}camera_optical"/>
-  </joint>
-<!-- ****************************************************** Camera Optical Link ******************************************************  -->
-  <link name="${prefix}camera_optical"/>
+    <xacro:include filename="${xacro_path}common_rviz_materials.xacro" />    <!--  RVIZ Colors  -->
+    <xacro:include filename="${xacro_path}rrbot_gz.xacro" />                 <!--  Gazebo Sim   -->
+    <xacro:include filename="${xacro_path}rrbot_r2c.xacro" />                <!--  ROS2_Control -->
+    <xacro:include filename="${xacro_path}rrbot_urdf.xacro" />               <!--  Robot URDF   -->
 <!-- ****************************************************** END **********************************************************************  -->
 </robot>

File: xacro/rrbot_r2c.xacro (robot description, xacro)
@@ -1,5 +1,5 @@
 <?xml version="1.0"?>
 <robot xmlns:xacro="http://www.ros.org/wiki/xacro">
-    <ros2_control name="rrbot" type="system">
+    <ros2_control name="rrbot_hw" type="system">
       <joint name="${prefix}joint1">
         <command_interface name="position">

Commit message: u

File: xacro/rrbot.xacro (robot description, xacro)
@@ -9,4 +9,5 @@
     <xacro:property name="mesh_path"    value="${pkg_path}/meshes/"     />
     <xacro:property name="xacro_path"   value="${pkg_path}/xacro/"      />
+    <xacro:property name="config_path"  value="${pkg_path}/config/"     />
     <xacro:property name="name_space"   value="rrbot" />
     <xacro:property name="prefix"       value=""      />

File: xacro/rrbot_gz.xacro (robot description, xacro)
@@ -37,5 +37,5 @@
   <gazebo>
     <plugin name="gz_ros2_control" filename="libgazebo_ros2_control.so">
-      <parameters>$(find robot_gazebo)/config/rrbot_forward_position.yaml</parameters>
+      <parameters>${config_path}rrbot_forward_position.yaml</parameters>
     </plugin>
   </gazebo>
