Commit message: u

File: xacro/rrbot_gz.xacro (robot description, xacro)
@@ -37,5 +37,5 @@
   <gazebo>
     <plugin name="gz_ros2_control" filename="libgazebo_ros2_control.so">
-      <parameters>${config_path}rrbot_forward_position.yaml</parameters>
+      <!-- <parameters>${config_path}rrbot_forward_position.yaml</parameters> -->
     </plugin>
   </gazebo>
@@ -91,4 +91,41 @@
     <material>Gazebo/Green</material>
   </gazebo>
+<!-- ****************************************************** hokuyo  ******************************************************************  -->
+  <gazebo reference="${prefix}hokuyo">
+    <sensor type="ray" name="head_hokuyo_sensor">
+      <plugin name="hokuyo" filename="libgazebo_ros_ray_sensor.so">
+        <ros>
+          <namespace>${name_space}</namespace>
+        </ros>
+        <output_type>sensor_msgs/LaserScan</output_type>
+      </plugin>
+      <update_rate>30</update_rate>
+      <pose>0 0 0 0 0 0</pose>
+      <visualize>false</visualize>
+      <ray>
+        <scan>
+          <horizontal>
+            <samples>720</samples>
+            <resolution>1</resolution>
+            <min_angle>-${radians(180)}</min_angle>
+            <max_angle> ${radians(180)}</max_angle>
+          </horizontal>
+        </scan>
+        <range>
+          <min>0.10</min>
+          <max>30.0</max>
+          <resolution>0.01</resolution>
+        </range>
+<!-- Noise parameters based on published spec for Hokuyo laser achieving "+-30mm" accuracy at range < 10m.  A mean of 0.0m and stddev   -->
+<!-- of 0.01m will put 99.7% of samples within 0.03m of the true reading.                                                               -->
+        <noise>
+          <type>gaussian</type>
+          <mean>0.0</mean>
+          <stddev>0.01</stddev>
+        </noise>
+      </ray>
+    </sensor>
+    <!-- <material>Gazebo/Red</material> -->
+  </gazebo>
 <!-- ****************************************************** END **********************************************************************  -->
 </robot>

File: xacro/rrbot_urdf.xacro (robot description, xacro)
@@ -169,4 +169,31 @@
 <!-- ****************************************************** Camera Optical Link ******************************************************  -->
   <link name="${prefix}camera_optical"/>
+<!-- ****************************************************** Hokuyo Joint *************************************************************  -->
+  <joint name="${prefix}hokuyo_joint" type="fixed">
+    <axis xyz="0 1 0" />
+    <origin xyz="0 0 ${hokuyo_z}" rpy="0 0 0"/>
+    <parent link="${prefix}link3"/>
+    <child link="${prefix}hokuyo"/>
+  </joint>
+<!-- ****************************************************** Hokuyo Link **************************************************************  -->
+  <link name="${prefix}hokuyo">
+    <collision>
+      <origin xyz="0 0 0" rpy="0 0 0"/>
+      <geometry>
+        <box size="${hokuyo_length} ${hokuyo_width} ${hokuyo_height}"/>
+      </geometry>
+    </collision>
+    <visual>
+      <origin xyz="0 0 0" rpy="0 0 0"/>
+      <geometry>
+         <mesh filename="${mesh_path}hokuyo.dae"/> <!-- <box size="${hokuyo_length} ${hokuyo_width} ${hokuyo_height}"/>  -->
+      </geometry>
+    </visual>
+    <inertial>
+      <mass value="${hokuyo_mass}" />
+      <origin xyz="0 0 0" rpy="0 0 0"/>
+      <inertia ixx="1e-6" ixy="0" ixz="0" iyy="1e-6" iyz="0" izz="1e-6" />
+    </inertial>
+  </link>
 <!-- ****************************************************** END **********************************************************************  -->
 </robot>
